Commit message: fix to vessel_v2.urdf to correctly visualize robot model in rviz2 interface

File: urdf/vessel_v2.urdf (robot description, URDF)
Before this commit: robot vessel_v2, 7 links, 6 joints
Links:
- link base_link: geometry collision box size=13.11 5.27 2.04; visual mesh filename=package://asv_simulator/models/vessel_v2/meshes/vessel_simp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 scale=0.0556 0.0556 0.0556
